Commit message: UKF con imu

File: src/my_robot_sim/resource/diff_drive.urdf (robot description, URDF)
Before this commit: robot diff_drive, 6 links, 5 joints
Links:
- added link imu_link, mass 0.001; collision box size=0.01 0.01 0.01; visual box size=0.01 0.01 0.01
Joints:
- added joint base_link_to_imu: type fixed, parent base_link, child imu_link, origin xyz=0 0 0.035 rpy=0 0 0
